Commit message: added rest of the thigs and modified the world file

File: simplebot_description/urdf/gazebo.xacro (robot description, xacro)
@@ -70,5 +70,5 @@
         </sensor>
     </gazebo>
-    <gazebo>
+    <!-- <gazebo>
         <plugin name="diff_drive" filename="libgazebo_ros_diff_drive.so">
             <left_joint>left_wheel_joint</left_joint>
@@ -88,15 +88,37 @@
             <max_wheel_acceleration>1.0</max_wheel_acceleration>
         </plugin>
-    </gazebo>
+    </gazebo> -->
+    <gazebo>
+        <plugin name='diff_drive' filename='libgazebo_ros_diff_drive.so'>
+            <ros>
+            <namespace>/</namespace>
+            </ros>
+            <!-- wheels -->
+            <left_joint>left_wheel_joint</left_joint>
+            <right_joint>right_wheel_joint</right_joint>
+            <!-- kinematics -->
+            <wheel_separation>0.34</wheel_separation>
+            <wheel_diameter>0.14</wheel_diameter>
+            <!-- limits -->
+            <max_wheel_torque>20</max_wheel_torque>
+            <max_wheel_acceleration>1.0</max_wheel_acceleration>
+            <!-- output -->
+            <publish_odom>true</publish_odom>
+            <publish_odom_tf>true</publish_odom_tf>
+            <publish_wheel_tf>true</publish_wheel_tf>
+            <odometry_frame>odom</odometry_frame>
+            <robot_base_frame>base_link</robot_base_frame>
+        </plugin>
+        </gazebo>
     <gazebo reference="lidar_link">
         <sensor name="lidar" type="ray">
             <always_on>true</always_on>
             <visualize>true</visualize>
-            <update_rate>5</update_rate>
+            <update_rate>10</update_rate>
             <ray>
                 <scan>
                     <horizontal>
                     <samples>360</samples>
-                    <resolution>1.000000</resolution>
+                    <resolution>0.500000</resolution>
                     <min_angle>0.000000</min_angle>
                     <max_angle>6.280000</max_angle>
@@ -104,5 +126,5 @@
                 </scan>
                 <range>
-                    <min>0.120000</min>
+                    <min>0.170000</min>
                     <max>3.5</max>
                     <resolution>0.015000</resolution>

File: simplebot_description/urdf/simple_bot.urdf.xacro (robot description, xacro)
@@ -26,5 +26,5 @@
         </collision>
         <inertial>
-            <mass value="0.5"/>
+            <mass value="1.0"/>
             <inertia ixx="0.001" ixy="0.0" ixz="0.0" iyy="0.001" iyz="0.0" izz="0.001"/>
         </inertial>
@@ -32,6 +32,6 @@
     <joint name="base_joint" type="fixed">
         <origin xyz="0.0 0.0 ${z_off}" rpy="0.0 0.0 0.0"/>
-        <parent link="base_footprint"/>
-        <child link="base_link"/>
+        <parent link="base_link"/>
+        <child link="base_footprint"/>
     </joint>
     <xacro:macro name="wheel_def" params="wheel_name direction">
@@ -51,6 +51,6 @@
             </collision>
             <inertial>
-                <mass value="1.0"/>
-                <inertia ixx="0.01" iyy="0.01" izz="0.01" ixy="0.0" ixz="0.0" iyz="0.0"/>
+                <mass value="0.5"/>
+                <inertia ixx="0.0001" iyy="0.0001" izz="0.0001" ixy="0.0" ixz="0.0" iyz="0.0"/>
             </inertial>
         </link>
